Commit message: try to work with real robot

File: urdf/threeDOF (copy).urdf (robot description, URDF)
Before this commit: robot threeDOF, 10 links, 9 joints
Links:
- added link link1sail; visual box size=0.04 0.1 0.1
- added link link2sail; visual box size=0.04 0.3 0.08
- added link link3sail; visual box size=0.03 0.25 0.06
- added link pitch1motor; visual cylinder length=0.4 radius=0.01
- added link pitch2motor; visual cylinder length=0.3 radius=0.008
- added link yawmotor; visual cylinder length=0.1 radius=0.2
- link link1bar: geometry visual cylinder length=0.2 radius=0.02
- link table: geometry visual box size=1.0 1.0 0.05
Joints:
- removed joint Thor/1
- removed joint Thor/2
- removed joint Thor/3
- added joint attach-link1sail: type fixed, parent link1, child link1sail
- added joint attach-link2sail: type fixed, parent link2, child link2sail
- added joint attach-link3sail: type fixed, parent link3, child link3sail
- added joint attach-pitch1motor: type fixed, parent link1, child pitch1motor
- added joint attach-pitch2motor: type fixed, parent link2, child pitch2motor
- added joint attach-yawmotor: type fixed, parent world, child yawmotor
- added joint theta1: type continuous, parent world, child link1, origin xyz=0 0 0 rpy=0 0 0, axis 0 0 1
- added joint theta2: type continuous, parent link1, child link2, origin xyz=0 0 0 rpy=0 0 0, axis 1 0 0
- added joint theta3: type continuous, parent link2, child link3, origin xyz=0 .167 0 rpy=0 0 0, axis 1 0 0

Commit message: added motors to urdf

File: urdf/threeDOF (copy).urdf (robot description, URDF)
Before this commit: robot threeDOF, 16 links, 15 joints
Links:
- link pitch1motor: geometry visual cylinder length=0.04 radius=0.01
- link table: geometry visual box size=.3 .3 0.05

File: urdf/threeDOF.urdf (robot description, URDF)
Before this commit: robot threeDOF, 10 links, 9 joints
Links:
- added link pitch1motor; visual cylinder length=0.05 radius=0.03
- added link pitch2motor; visual cylinder length=0.05 radius=0.03
- added link yawmotor; visual cylinder length=0.05 radius=0.03
- link table: geometry visual box size=.3 .3 0.00635
Joints:
- added joint attach-pitch1motor: type fixed, parent link2, child pitch1motor
- added joint attach-pitch2motor: type fixed, parent link3, child pitch2motor
- added joint attach-yawmotor: type fixed, parent link1, child yawmotor
