Commit message: Refactor everythinggit add urdf/threeDOF\(depracated\).urdf !

File: urdf/threeDOF(depracated).urdf (robot description, URDF)
Before this commit: robot threeDOF, 13 links, 12 joints
Joints:
- joint Thor/1: origin xyz=-0.005 0.217 0 rpy=0 0 0 -> xyz=0 0 0 rpy=0 0 0
- joint Thor/2: origin xyz=0 0 .078 rpy=0 0 0 -> xyz=0 0 .09 rpy=0 0 0

File: urdf/threeDOF.urdf (robot description, URDF)
Before this commit: robot threeDOF, 13 links, 12 joints
Joints:
- joint Thor/1: origin xyz=0 0 0 rpy=0 0 0 -> xyz=-0.052 -0.2125 0 rpy=0 0 0
- joint Thor/2: origin xyz=0 0 .09 rpy=0 0 0 -> xyz=0 0 .085 rpy=0 0 0
- joint Thor/3: origin xyz=-.03 .167 0 rpy=0 0 0 -> xyz=-.0368 .1651 0 rpy=0 0 0
- joint shifttotip: origin xyz=0 .252 0 rpy=0 0 0 -> xyz=0 .2522 0 rpy=0 0 0
