Commit message: fixed urdf, added SinTraj class, sin motion working

File: urdf/threeDOF.urdf (robot description, URDF)
Before this commit: robot threeDOF, 16 links, 15 joints
Links:
- link link3bar: geometry visual cylinder length=1 radius=0.02

Commit message: Made the plots work

File: urdf/threeDOF.urdf (robot description, URDF)
Before this commit: robot threeDOF, 13 links, 12 joints
Joints:
- joint Thor/2: axis -1 0 0 -> 1 0 0
- joint Thor/3: axis 1 0 0 -> -1 0 0; origin xyz=0 .167 0 rpy=0 0 0 -> xyz=-.03 .167 0 rpy=0 0 0

Commit message: touch_points was working momentarily, grav compensated

File: urdf/threeDOF.urdf (robot description, URDF)
Before this commit: robot threeDOF, 13 links, 12 joints
Joints:
- joint shifttotip: origin xyz=0 .254 0 rpy=0 0 0 -> xyz=0 .252 0 rpy=0 0 0

File: urdf/threeDOF_table.urdf (robot description, URDF)
Before this commit: robot threeDOF, 16 links, 15 joints
Links:
- removed link link1sail
- removed link link2sail
- removed link link3sail
- link link1bar: geometry visual cylinder length=.09 radius=0.02
- link pitch1motor: geometry visual cylinder length=0.05 radius=0.03
- link pitch2motor: geometry visual cylinder length=0.05 radius=0.03
- link table: geometry visual box size=.3 .3 0.00635
- link yawmotor: geometry visual cylinder length=0.05 radius=0.03
Joints:
- removed joint attach-link1sail
- removed joint attach-link2sail
- removed joint attach-link3sail
- removed joint theta1
- removed joint theta2
- removed joint theta3
- added joint Thor/1: type continuous, parent world, child link1, origin xyz=-0.005 0.217 0 rpy=0 0 0, axis 0 0 1
- added joint Thor/2: type continuous, parent link1, child link2, origin xyz=0 0 .078 rpy=0 0 0, axis 1 0 0
- added joint Thor/3: type continuous, parent link2, child link3, origin xyz=-.03 .167 0 rpy=0 0 0, axis -1 0 0
- joint attach-pitch1motor: parent link1 -> link2
- joint attach-pitch2motor: parent link2 -> link3
- joint attach-yawmotor: parent world -> link1
- joint shifttotip: origin xyz=0 .254 0 rpy=0 0 0 -> xyz=0 .252 0 rpy=0 0 0

Commit message: Make faster, hopefully

File: urdf/threeDOF.urdf (robot description, URDF)
Before this commit: robot threeDOF, 13 links, 12 joints
Joints:
- removed joint Thor/2
- added joint Thor/4: type continuous, parent link1, child link2, origin xyz=0 0 .085 rpy=0 0 0, axis 1 0 0

Commit message: updated 3dof urdf, added undistortion

File: urdf/threeDOF.urdf (robot description, URDF)
Before this commit: robot threeDOF, 13 links, 12 joints
Joints:
- joint Thor/3: origin xyz=-.0368 .1651 0 rpy=0 0 0 -> xyz=-.0368 .2794 0 rpy=0 0 0
- joint shifttotip: origin xyz=0 .2522 0 rpy=0 0 0 -> xyz=-.0368 .303993 0 rpy=0 0 0

Commit message: Make detector better

File: urdf/threeDOF.urdf (robot description, URDF)
Before this commit: robot threeDOF, 13 links, 12 joints
Joints:
- removed joint Thor/4
- added joint Thor/6: type continuous, parent link1, child link2, origin xyz=0 0 .085 rpy=0 0 0, axis 1 0 0

Commit message: Add map to rviz

File: urdf/threeDOF.urdf (robot description, URDF)
Before this commit: robot threeDOF, 13 links, 12 joints
Links:
- added link map
Joints:
- added joint world_to_map: type fixed, parent world, child map, origin xyz=0 0 0 rpy=0 0 0
- joint Thor/6: origin xyz=0 0 .085 rpy=0 0 0 -> xyz=0.00695 0 .085 rpy=0 0 0
- joint shifttotip: origin xyz=-.0368 .303993 0 rpy=0 0 0 -> xyz=0 .303993 0 rpy=0 0 0
