Commit message: visuals approx right

File: urdf/fiveDOF.urdf (robot description, URDF)
Before this commit: robot threeDOF, 15 links, 14 joints
Joints:
- removed joint Thor/2
- added joint Thor/6: type continuous, parent link1, child link2, origin xyz=0 0 .085 rpy=0 0 0, axis 1 0 0

File: urdf/threeDOF.urdf (robot description, URDF)
Before this commit: robot threeDOF, 13 links, 12 joints
Links:
- link link2bar: geometry visual cylinder length=.3 radius=0.02
- link link3bar: geometry visual cylinder length=.35 radius=0.02

Commit message: added 5dof functionality

File: urdf/fiveDOF.urdf (robot description, URDF)
Before this commit: robot fiveDOF, 15 links, 14 joints
Links:
- added link link4bar; visual cylinder length=.1 radius=0.02
- added link map
- added link pitch3motor; visual cylinder length=0.05 radius=0.03
- added link pitch4motor; visual cylinder length=0.05 radius=0.03
Joints:
- added joint attach-link4bar: type fixed, parent link4, child link4bar
- added joint attach-pitch3motor: type fixed, parent link4, child pitch3motor
- added joint attach-pitch4motor: type fixed, parent link5, child pitch4motor
- added joint world_to_map: type fixed, parent world, child map, origin xyz=0 0 0 rpy=0 0 0
- joint Thor/3: origin xyz=-.0368 .1651 0 rpy=0 0 0 -> xyz=-.0368 .2794 0 rpy=0 0 0
- joint Thor/4: origin xyz=-.0368 .1651 0 rpy=0 0 0 -> xyz=0 .303993 0 rpy=0 0 0
- joint Thor/5: axis -1 0 0 -> 0 0 1; origin xyz=-.0368 .1651 0 rpy=0 0 0 -> xyz=-.05 0 -.05 rpy=0 0 0
- joint Thor/6: origin xyz=0 0 .085 rpy=0 0 0 -> xyz=0.00695 0 .085 rpy=0 0 0
- joint shifttotip: origin xyz=0 .2522 0 rpy=0 0 0 -> xyz=0 0 -.05 rpy=0 0 0

Commit message: 5DOF

File: urdf/fiveDOF.urdf (robot description, URDF)
Before this commit: robot fiveDOF, 19 links, 18 joints
Joints:
- removed joint Thor/5
- added joint Thor/2: type continuous, parent link4, child link5, origin xyz=.05 0 -.05 rpy=0 0 0, axis 0 0 -1
- joint Thor/4: axis -1 0 0 -> 1 0 0

Commit message: configured gravity, urdf accurate

File: urdf/fiveDOF.urdf (robot description, URDF)
Before this commit: robot fiveDOF, 19 links, 18 joints
Joints:
- joint Thor/2: origin xyz=.05 0 -.05 rpy=0 0 0 -> xyz=-.05 0 -.05 rpy=0 0 0
